File: Circuit/V1/MotorDriver_V1_1/MotorDriver_V1_1.kicad_sch (KiCad schematic)
At the start: 0 parts

Commit message: MD完成
Parts:
- added C1, C2: 0.1u, Capacitor_SMD:C_0603_1608Metric_Pad1.08x0.95mm_HandSolder, symbol Device:C
- added C3, C4, C5, C6: 10u, Capacitor_SMD:C_0805_2012Metric_Pad1.18x1.45mm_HandSolder, symbol Device:C
- added H1, H2: MountingHole, MountingHole:MountingHole_3.2mm_M3_Pad_Via, symbol Mechanical:MountingHole
- added J1: Conn_01x04, Connector_JST:JST_XH_B4B-XH-A_1x04_P2.50mm_Vertical, symbol Connector_Generic:Conn_01x04
- added J2, J3: Conn_01x06_Pin, Connector_PinHeader_2.54mm:PinHeader_1x06_P2.54mm_Vertical, symbol Connector:Conn_01x06_Pin
- added J4, J5, J6: Conn_01x02, Connector_JST:JST_XH_B2B-XH-A_1x02_P2.50mm_Vertical, symbol Connector_Generic:Conn_01x02
- added U1, U2: AM2837, Package_SO:SOP-8_3.76x4.96mm_P1.27mm, symbol 0-Library:AM2837
Connections:
- new net GND: C3.1, C4.1, C5.1, C6.1, J2.1 (Pin_1), J3.1 (Pin_1), J5.1 (Pin_1), U1.3 (GND), U2.3 (GND)
- new net IN1A: J1.4 (Pin_4), J2.5 (Pin_5), U1.1 (INA)
- new net IN1B: J1.3 (Pin_3), J2.4 (Pin_4), U1.2 (INB)
- new net IN2A: J1.2 (Pin_2), J2.2 (Pin_2), U2.1 (INA)
- new net IN2B: J1.1 (Pin_1), J2.3 (Pin_3), U2.2 (INB)
- new net OUT1A: C1.2, J3.2 (Pin_2), J4.2 (Pin_2), U1.7 (OUTA), U1.8 (OUTA)
- new net OUT1B: C1.1, J3.3 (Pin_3), J4.1 (Pin_1), U1.5 (OUTB), U1.6 (OUTB)
- new net OUT2A: C2.2, J3.5 (Pin_5), J6.1 (Pin_1), U2.7 (OUTA), U2.8 (OUTA)
- new net OUT2B: C2.1, J3.4 (Pin_4), J6.2 (Pin_2), U2.5 (OUTB), U2.6 (OUTB)
- new net VCC: C3.2, C4.2, C5.2, C6.2, J2.6 (Pin_6), J3.6 (Pin_6), J5.2 (Pin_2), U1.4 (VCC), U2.4 (VCC)
