File: Circuit/V1/MotorDriver_V1_1/MotorDriver_V1_1.kicad_sch (KiCad schematic)
At the start: 16 parts, among them J1 Conn_01x04, J2 Conn_01x06_Pin, J3 Conn_01x06_Pin, J4 Conn_01x02, J5 Conn_01x02, J6 Conn_01x02, U1 AM2837, U2 AM2837

Commit message: 発注
Parts:
- added C7: 10u, Capacitor_SMD:C_0805_2012Metric_Pad1.18x1.45mm_HandSolder, symbol Device:C
Connections:
- net GND: now also C7.1
- net VCC: now also C7.2
Changed lines of the file:
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@@
+	)
+	(junction
+		(at 33.02 68.58)
+		(diameter 0)
+		(color 0 0 0 0)
 	)
 	(junction
@@
 	)
 	(junction
+		(at 25.4 58.42)
+		(diameter 0)
+		(color 0 0 0 0)
+	)
+	(junction
 		(at 33.02 48.26)
 		(diameter 0)
@@
 	(wire
 		(pts
+			(xy 33.02 68.58) (xy 33.02 73.66)
+		)
+		(stroke
+			(width 0)
+			(type default)
+		)
+	)
+	(wire
+		(pts
 			(xy 53.34 35.56) (xy 53.34 38.1)
 		)
@@
 	(wire
 		(pts
-			(xy 33.02 58.42) (xy 33.02 63.5)
+			(xy 33.02 58.42) (xy 33.02 68.58)
 		)
 		(stroke
@@
 		(pts
 			(xy 87.63 48.26) (xy 87.63 58.42)
+		)
+		(stroke
+			(width 0)
+			(type default)
+		)
+	)
+	(wire
+		(pts
+			(xy 25.4 58.42) (xy 25.4 68.58)
 		)
 		(stroke
@@
 				(path "/83381d65-5a20-4ed4-8930-66ed727b8ae3"
 					(reference "#PWR05")
+					(unit 1)
+				)
+			)
+		)
+	)
+	(symbol
+		(lib_id "Device:C")
+		(at 29.21 68.58 270)
+		(unit 1)
+		(exclude_from_sim no)
+		(in_bom yes)
+		(on_board yes)
+		(dnp no)
+		(property "Reference" "C7"
+			(at 29.21 64.77 90)
+			(effects
+				(font
+					(size 1.27 1.27)
+				)
+			)
+		)
+		(property "Value" "10u"
+			(at 29.21 72.39 90)
+			(effects
+				(font
+					(size 1.27 1.27)
+				)
+			)
+		)
+		(property "Footprint" "Capacitor_SMD:C_0805_2012Metric_Pad1.18x1.45mm_HandSolder"
+			(at 25.4 69.5452 0)
+			(effects
+				(font
+					(size 1.27 1.27)
+				)
+				(hide yes)
+			)
+		)
+		(property "Datasheet" "~"
+			(at 29.21 68.58 0)
+			(effects
+				(font
+					(size 1.27 1.27)
+				)
+				(hide yes)
+			)
+		)
+		(property "Description" "Unpolarized capacitor"
+			(at 29.21 68.58 0)
+			(effects
+				(font
+					(size 1.27 1.27)
+				)
+				(hide yes)
+			)
+		)
+		(pin "1"
+		)
+		(pin "2"
+		)
+		(instances
+			(project "MotorDriver_V1_1"
+				(path "/83381d65-5a20-4ed4-8930-66ed727b8ae3"
+					(reference "C7")
 					(unit 1)
 				)
@@
 	(symbol
 		(lib_id "power:GND")
-		(at 33.02 63.5 0)
+		(at 33.02 73.66 0)
 		(unit 1)
 		(exclude_from_sim no)
@@
 		(dnp no)
 		(property "Reference" "#PWR06"
-			(at 33.02 69.85 0)
+			(at 33.02 80.01 0)
 			(effects
 				(font
@@
 		)
 		(property "Value" "GND"
-			(at 33.02 67.31 0)
+			(at 33.02 77.47 0)
 			(effects
 				(font
@@
 		)
 		(property "Footprint" ""
-			(at 33.02 63.5 0)
+			(at 33.02 73.66 0)
 			(effects
 				(font
@@
 		)
 		(property "Datasheet" ""
-			(at 33.02 63.5 0)
+			(at 33.02 73.66 0)
 			(effects
 				(font
@@
 		)
 		(property "Description" "Power symbol creates a global label with name \"GND\" , ground"
-			(at 33.02 63.5 0)
-			(effects
-				(font
+			(at 33.02 73.66 0)
+			(effects
+				(font
