File: Circuit/MainBoard/MainBoard_V1_1/MainBoard_V1_1.kicad_sch (KiCad schematic)
At the start: 56 parts, among them J1 Conn_01x17_Socket, J10 Conn_01x04, J11 Conn_01x04, J12 Conn_01x04, J13 Conn_01x04, J2 Conn_01x17_Socket, J3 Conn_01x02, J4 Conn_01x02, J5 Conn_01x02, J6 Conn_01x03, J7 Conn_01x03, J8 Conn_01x03, J9 Conn_01x04, Q1 Q_PMOS_GDS, SW1 SW_Push_Dual, SW2 SW_Slide_DPDT, SW3 SW_Push_Dual, SW4 SW_Push_Dual, U1 BP5293-33, U2 RP2040

Commit message: 進捗
Parts:
- removed U1: BP5293-33, 0-Library:BP5293-33, symbol 0-Library:BP5293-33
- added J17, J18: Conn_01x03, Connector_JST:JST_XH_B3B-XH-A_1x03_P2.50mm_Vertical, symbol Connector_Generic:Conn_01x03
- added R13, R14: 10k, Resistor_THT:R_Axial_DIN0207_L6.3mm_D2.5mm_P10.16mm_Horizontal, symbol Device:R
- added U1: LM1117MP-3.3, Package_TO_SOT_SMD:SOT-223-3_TabPin2, symbol Regulator_Linear:LM1117MP-3.3
- gave numbers to parts that had none: 3
- renumbered J13 to J10, J6 to J11, J7 to J12, J8 to J13, J9 to J6, J10 to J7, J11 to J8, J12 to J9
Connections:
- net +3V3: now also J17.2 (Pin_2), J18.2 (Pin_2), R13.1, R14.1, U1.2 (VO)
- net GND: now also J17.1 (Pin_1), J18.1 (Pin_1), U1.1 (GND)
- net M1A: now also J2.7 (Pin_7), J9.1 (Pin_1), U2.28 (25); no longer J9.4 (Pin_4)
- net M1B: now also J2.8 (Pin_8), J9.2 (Pin_2), U2.27 (24); no longer J9.3 (Pin_3)
- net M2A: now also J2.9 (Pin_9), J9.3 (Pin_3), U2.26 (23); no longer J9.2 (Pin_2)
- net M2B: now also J2.10 (Pin_10), J9.4 (Pin_4), U2.25 (22); no longer J9.1 (Pin_1)
- net M3A: now also J10.1 (Pin_1), J2.11 (Pin_11), U2.24 (21); no longer J10.4 (Pin_4)
- net M3B: now also J10.2 (Pin_2), J2.12 (Pin_12), U2.23 (20); no longer J10.3 (Pin_3)
- net M4A: now also J10.3 (Pin_3), J2.13 (Pin_13), U2.22 (19); no longer J10.2 (Pin_2)
- net M4B: now also J10.4 (Pin_4), J2.14 (Pin_14), U2.21 (18); no longer J10.1 (Pin_1)
- net SCL: now also R14.2
- net SDA: now also R13.2
- net VCC: now also U1.3 (VI)
- new net GPIO3: J17.3 (Pin_3)
- new net GPIO4: J18.3 (Pin_3)
Other:
- moved on the sheet: H1, H2, H3, H4, J10, J11, J12, J13, J14, J15, J16, J3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

Commit message: 発注
Parts:
- added BZ1: Buzzer, Buzzer_Beeper:Buzzer_TDK_PS1240P02BT_D12.2mm_H6.5mm, symbol Device:Buzzer
- added C9: 0.1u, Capacitor_THT:C_Disc_D3.0mm_W1.6mm_P2.50mm, symbol Device:C
- added Q2: DTC114E, symbol Transistor_BJT:DTC114E
- added R15: 1k, Resistor_THT:R_Axial_DIN0207_L6.3mm_D2.5mm_P10.16mm_Horizontal, symbol Device:R
- added TP1, TP2: TestPoint, TestPoint:TestPoint_THTPad_D1.5mm_Drill0.7mm, symbol Connector:TestPoint
- R1, R11, R4, R6, R9: value 10k -> 1k
- R8: value 1k -> 10k
Connections:
- net +3V3: now also TP2.1
- net GND: now also C9.1, Q2.2 (E)
- net GPIO0: now also J1.16 (Pin_16), U2.16 (14)
- net GPIO1: now also J1.15 (Pin_15), U2.15 (13)
- net GPIO2: now also J1.12 (Pin_12), U2.12 (10)
- net GPIO3: now also J1.5 (Pin_5), U2.5 (3)
- net GPIO4: now also J1.4 (Pin_4), U2.4 (2)
- net LED1: now also J1.8 (Pin_8), U2.8 (6)
- net LED2: now also J1.13 (Pin_13), U2.13 (11)
- net LED3: now also J1.9 (Pin_9), U2.9 (7)
- net LED4: now also J1.14 (Pin_14), U2.14 (12)
- net SW1: now also J1.10 (Pin_10), U2.10 (8)
- net SW2: now also J2.15 (Pin_15), U2.20 (17)
- net SW3: now also J2.16 (Pin_16), U2.19 (16)
- net VCC: now also BZ1.1 (+), C9.2, R15.1, TP1.1
- net BUZZER: now reaches J1.17 (Pin_17), U2.17 (15)
- net BUZZER: now also Q2.1 (B)
- new net: BZ1.2 (-), Q2.3 (C), R15.2

Commit message: 最終修正
Parts:
- BZ1: value Buzzer -> PKM13EPYH4000-A0
- Q1: value Q_PMOS_GDS -> TJ60S04M3L
- SW1, SW3, SW4: value SW_Push_Dual -> TVGP01-G73BB
- SW2: value SW_Slide_DPDT -> IS-2235
Other:
- note added: "Buzzer"
- note added: "Connectors"
- moved on the sheet: BZ1, C9, H1, H2, H3, H4, Q2, R15, TP1, TP2

Commit message: 最終発注
Parts:
- R12, R7: value 10k -> 1k
Connections:
- net GPIO0 renamed GPIOA
- net GPIO1 renamed GPIOB
- net GPIO2 renamed GPIOC
- net GPIO3 renamed GPIOD
- net GPIO4 renamed GPIOE
Changed lines of the file:
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@@
 		)
 	)
-	(global_label "GPIO1"
+	(global_label "GPIOB"
 		(shape bidirectional)
 		(at 113.03 146.05 90)
@@
 		)
 		(property "Intersheetrefs" "${INTERSHEET_REFS}"
-			(at 113.03 136.2687 90)
+			(at 113.03 136.2082 90)
 			(effects
 				(font
@@
 		)
 	)
-	(global_label "GPIO2"
+	(global_label "GPIOC"
 		(shape bidirectional)
 		(at 132.08 146.05 90)
@@
 		)
 		(property "Intersheetrefs" "${INTERSHEET_REFS}"
-			(at 132.08 136.2687 90)
+			(at 132.08 136.2082 90)
 			(effects
 				(font
@@
 		)
 	)
-	(global_label "GPIO0"
+	(global_label "GPIOA"
 		(shape bidirectional)
 		(at 93.98 146.05 90)
@@
 		)
 		(property "Intersheetrefs" "${INTERSHEET_REFS}"
-			(at 93.98 136.2687 90)
+			(at 93.98 136.3896 90)
 			(effects
 				(font
@@
 		)
 	)
-	(global_label "GPIO2"
+	(global_label "GPIOC"
 		(shape bidirectional)
 		(at 157.48 67.31 180)
@@
 		)
 		(property "Intersheetrefs" "${INTERSHEET_REFS}"
-			(at 147.6987 67.31 0)
+			(at 147.6382 67.31 0)
 			(effects
 				(font
@@
 		)
 	)
-	(global_label "GPIO1"
+	(global_label "GPIOB"
 		(shape bidirectional)
 		(at 157.48 74.93 180)
@@
 		)
 		(property "Intersheetrefs" "${INTERSHEET_REFS}"
-			(at 147.6987 74.93 0)
+			(at 147.6382 74.93 0)
 			(effects
 				(font
@@
 		)
 	)
-	(global_label "GPIO3"
+	(global_label "GPIOD"
 		(shape bidirectional)
 		(at 151.13 146.05 90)
@@
 		)
 		(property "Intersheetrefs" "${INTERSHEET_REFS}"
-			(at 151.13 136.2687 90)
+			(at 151.13 136.2082 90)
 			(effects
 				(font
@@
 		)
 	)
-	(global_label "GPIO4"
+	(global_label "GPIOE"
 		(shape bidirectional)
 		(at 157.48 46.99 180)
@@
 		)
 		(property "Intersheetrefs" "${INTERSHEET_REFS}"
-			(at 147.6987 46.99 0)
+			(at 147.7592 46.99 0)
 			(effects
 				(font
@@
 		)
 	)
-	(global_label "GPIO3"
+	(global_label "GPIOD"
 		(shape bidirectional)
 		(at 157.48 49.53 180)
@@
 		)
 		(property "Intersheetrefs" "${INTERSHEET_REFS}"
-			(at 147.6987 49.53 0)
+			(at 147.6382 49.53 0)
 			(effects
 				(font
@@
 		)
 	)
-	(global_label "GPIO4"
+	(global_label "GPIOE"
 		(shape bidirectional)
 		(at 170.18 146.05 90)
@@
 		)
 		(property "Intersheetrefs" "${INTERSHEET_REFS}"
-			(at 170.18 136.2687 90)
+			(at 170.18 136.3292 90)
 			(effects
 				(font
@@
 		)
 	)
-	(global_label "GPIO0"
+	(global_label "GPIOA"
 		(shape bidirectional)
 		(at 157.48 77.47 180)
@@
 		)
 		(property "Intersheetrefs" "${INTERSHEET_REFS}"
-			(at 147.6987 77.47 0)
+			(at 147.8196 77.47 0)
 			(effects
 				(font
@@
 			)
 		)
-		(property "Value" "10k"
+		(property "Value" "1k"
 			(at 74.93 82.55 90)
 			(effects
@@
 			)
 		)
-		(property "Value" "10k"
+		(property "Value" "1k"
 			(at 74.93 69.85 90)
 			(effects
