File: Circuit/MainBoard/MainBoard_V1_1/MainBoard_V1_1.kicad_pcb (KiCad board)
At the start: 2 copper layers, 70 x 70 mm, 53 parts, among them J1 Conn_01x17_Socket, J10 Conn_01x04, J11 Conn_01x04, J12 Conn_01x04, J13 Conn_01x04, J2 Conn_01x17_Socket, J3 Conn_01x02, J4 Conn_01x02, J5 Conn_01x02, J6 Conn_01x03, J7 Conn_01x03, J8 Conn_01x03, J9 Conn_01x04, Q1 Q_PMOS_GDS, SW1 SW_Push_Dual, SW2 SW_Slide_DPDT, SW3 SW_Push_Dual, SW4 SW_Push_Dual, U1 BP5293-33, U2 RP2040

Commit message: 進捗
Parts:
- added J14: Conn_01x03, Connector_JST:JST_XH_B3B-XH-A_1x03_P2.50mm_Vertical, F.Cu at (-31.0, 22.5)
- added J15: Conn_01x03, Connector_JST:JST_XH_B3B-XH-A_1x03_P2.50mm_Vertical, F.Cu at (-31.0, 12.5)
- added J16: Conn_01x03, Connector_JST:JST_XH_B3B-XH-A_1x03_P2.50mm_Vertical, F.Cu at (-31.0, 2.50)
- added J17: Conn_01x03, Connector_JST:JST_XH_B3B-XH-A_1x03_P2.50mm_Vertical, F.Cu at (-31.0, -7.50)
- added J18: Conn_01x03, Connector_JST:JST_XH_B3B-XH-A_1x03_P2.50mm_Vertical, F.Cu at (-31.0, -17.5)
- added R13: 10k, Resistor_THT:R_Axial_DIN0207_L6.3mm_D2.5mm_P10.16mm_Horizontal, F.Cu at (5.08, -21.0)
- added R14: 10k, Resistor_THT:R_Axial_DIN0207_L6.3mm_D2.5mm_P10.16mm_Horizontal, F.Cu at (5.08, -17.8)
- J11, J12, J13: value Conn_01x04 -> Conn_01x03; footprint Connector_JST:JST_XH_B4B-XH-A_1x04_P2.50mm_Vertical -> Connector_JST:JST_XH_B3B-XH-A_1x03_P2.50mm_Vertical
- J6, J7, J8: value Conn_01x03 -> Conn_01x04; footprint Connector_JST:JST_XH_B3B-XH-A_1x03_P2.50mm_Vertical -> Connector_JST:JST_XH_B4B-XH-A_1x04_P2.50mm_Vertical
- U1: value BP5293-33 -> LM1117MP-3.3; footprint 0-Library:BP5293-33 -> Package_TO_SOT_SMD:SOT-223-3_TabPin2; moved to B.Cu
- moved J13 65.9 mm to (31.0, -22.5), turned to -90 degrees
- moved J12 64.8 mm to (31.0, -12.5), turned to -90 degrees
- moved J11 63.5 mm to (31.0, -2.50), turned to -90 degrees
- moved J10 49.0 mm to (17.0, -16.5)
- moved J9 49.0 mm to (17.0, -22.5)
- moved J7 44.3 mm to (-24.5, -10.5)
- moved J8 44.3 mm to (-24.5, -16.5)
- moved J6 41.6 mm to (-24.5, -22.5)
- moved J4 35.5 mm to (28.5, 15.5)
- moved J5 35.5 mm to (28.5, 21.5)
- moved C2 27.4 mm to (17.8, -11.5), turned to 0 degrees
- moved R9 23.6 mm to (5.08, -24.2), turned to 180 degrees
- moved C6 23.3 mm to (25.2, 1.25), turned to 180 degrees
- moved C7 22.3 mm to (15.0, -28.2)
- moved C8 19.5 mm to (25.2, 6.75), turned to 180 degrees
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Connections:
- J1 pad 1: Net-(J1-Pin_1) -> unconnected-(J1-Pin_1-Pad1)
- J10 pad 1: GND -> M3A
- J10 pad 2: +3V3 -> M3B
- J10 pad 3: SDA -> M4A
- J10 pad 4: SCL -> M4B
- J11 pad 3: SDA -> ADC0
- J12 pad 1: M2B -> GND
- J12 pad 2: M2A -> +3V3
- J12 pad 3: M1B -> ADC1
- J13 pad 1: M4B -> GND
- J13 pad 2: M4A -> +3V3
- J13 pad 3: M3B -> ADC2
- J2 pad 10: Net-(J2-Pin_10) -> M2B
- J2 pad 11: Net-(J2-Pin_11) -> M3A
- J2 pad 12: Net-(J2-Pin_12) -> M3B
- J2 pad 13: Net-(J2-Pin_13) -> M4A
- J2 pad 14: Net-(J2-Pin_14) -> M4B
- J2 pad 7: Net-(J2-Pin_7) -> M1A
- J2 pad 8: Net-(J2-Pin_8) -> M1B
- J2 pad 9: Net-(J2-Pin_9) -> M2A
- J6 pad 3: ADC0 -> UART0_TX
- J7 pad 3: ADC1 -> SDA
- J8 pad 3: ADC2 -> SDA
- J9 pad 1: GND -> M1A
- J9 pad 2: +3V3 -> M1B
- J9 pad 3: UART0_TX -> M2A
- J9 pad 4: UART0_RX -> M2B
- U1 pad 1: VCC -> GND
- U1 pad 2: GND -> +3V3
- U1 pad 3: +3V3 -> VCC
- U2 pad 1: Net-(J1-Pin_1) -> unconnected-(J1-Pin_1-Pad1)
- U2 pad 21: Net-(J2-Pin_14) -> M4B
- U2 pad 22: Net-(J2-Pin_13) -> M4A
- U2 pad 23: Net-(J2-Pin_12) -> M3B
- U2 pad 24: Net-(J2-Pin_11) -> M3A
- U2 pad 25: Net-(J2-Pin_10) -> M2B
- U2 pad 26: Net-(J2-Pin_9) -> M2A
- U2 pad 27: Net-(J2-Pin_8) -> M1B
- U2 pad 28: Net-(J2-Pin_7) -> M1A
Routing:
- net +3V3: track 0.00 -> 261.0 mm
- net ADC0: track 0.00 -> 40.2 mm
- net ADC3: track 0.00 -> 35.8 mm
- net ADC1: track 0.00 -> 31.7 mm
- net GPIO0: track 0.00 -> 31.3 mm
- net M4B: track 0.00 -> 26.5 mm
- net ADC2: track 0.00 -> 25.8 mm
- net GPIO1: track 0.00 -> 23.9 mm
- net M2B: track 0.00 -> 22.5 mm
- net M4A: track 0.00 -> 21.9 mm
- net SDA: track 0.00 -> 21.8 mm
- net GPIO2: track 0.00 -> 20.9 mm
- net GPIO3: track 0.00 -> 19.1 mm
- net SCL: track 0.00 -> 18.4 mm
- net M2A: track 0.00 -> 17.9 mm
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- added copper zone on B.Cu, net +BATT
- added copper zone on F.Cu, net +BATT
- added copper zone on B.Cu, net Net-(D3-K)
- added copper zone on F.Cu, net Net-(D3-K)
- added copper zone on B.Cu, net VCC
- added copper zone on F.Cu, net VCC
Other:
- board text added: "ADC2"

Commit message: 発注
Parts:
- added ?: , , F.Cu at (-15.0, -28.8)
- added ?: , , F.Cu at (-20.0, -33.8)
- added ?: , , F.Cu at (-22.5, -31.2)
- added ?: , , F.Cu at (-15.0, -33.8)
- added ?: , , F.Cu at (-15.0, -31.2)
- added ?: , , F.Cu at (-22.5, -28.8)
- added ?: , , F.Cu at (-17.5, -28.8)
- added ?: , , F.Cu at (-25.0, -33.8)
- added ?: , , F.Cu at (-20.0, -31.2)
- added ?: , , F.Cu at (-25.0, -31.2)
- added ?: , , F.Cu at (-22.5, -33.8)
- added ?: , , F.Cu at (-25.0, -28.8)
- added ?: , , F.Cu at (-17.5, -33.8)
- added ?: , , F.Cu at (-17.5, -31.2)
- added ?: , , F.Cu at (-20.0, -28.8)
- added BZ1: Buzzer, Buzzer_Beeper:Buzzer_TDK_PS1240P02BT_D12.2mm_H6.5mm, F.Cu at (-18.0, 2.00)
- added C9: 0.1u, Capacitor_THT:C_Disc_D3.0mm_W1.6mm_P2.50mm, F.Cu at (-17.2, 15.8)
- added Q2: DTC114E, Package_TO_SOT_THT:TO-92_Inline, F.Cu at (-21.6, 16.3)
- added R15: 1k, Resistor_THT:R_Axial_DIN0207_L6.3mm_D2.5mm_P10.16mm_Horizontal, F.Cu at (-15.4, 10.2)
- added TP1: TestPoint, TestPoint:TestPoint_THTPad_D1.5mm_Drill0.7mm, F.Cu at (12.5, 14.2)
- added TP2: TestPoint, TestPoint:TestPoint_THTPad_D1.5mm_Drill0.7mm, F.Cu at (12.5, 16.8)
- R1, R11, R4, R6, R9: value 10k -> 1k
- R8: value 1k -> 10k
- moved R12 83.7 mm to (5.08, -28.2), turned to 180 degrees
- moved D8 79.3 mm to (18.8, -30.7), turned to 90 degrees
- moved D6 74.4 mm to (23.2, -30.7), turned to 90 degrees
- moved R7 52.4 mm to (5.25, -4.67), turned to 90 degrees
- moved R2 35.0 mm to (1.75, -14.8), turned to -90 degrees
- moved R10 19.8 mm to (5.25, -2.08), turned to -90 degrees
- moved R6 19.6 mm to (-1.75, -14.8), turned to -90 degrees
- moved R5 18.8 mm to (1.75, -2.08), turned to -90 degrees
- moved R1 15.3 mm to (-5.25, -14.8), turned to -90 degrees
- moved SW1 13.5 mm to (-21.5, 32.8), turned to 90 degrees
- moved SW3 13.5 mm to (-8.50, 32.8), turned to 90 degrees
- moved R11 11.4 mm to (-1.75, -2.08), turned to -90 degrees
- moved R4 10.5 mm to (-5.25, -2.08), turned to -90 degrees
- moved D7 4.95 mm to (1.50, 16.8)
- moved D5 4.61 mm to (-3.50, 16.8)
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Connections:
- net Net-(J1-Pin_17) renamed BUZZER
- J1 pad 10: Net-(J1-Pin_10) -> SW1
- J1 pad 12: Net-(J1-Pin_12) -> GPIO2
- J1 pad 13: Net-(J1-Pin_13) -> LED2
- J1 pad 14: Net-(J1-Pin_14) -> LED4
- J1 pad 15: Net-(J1-Pin_15) -> GPIO1
- J1 pad 16: Net-(J1-Pin_16) -> GPIO0
- J1 pad 4: Net-(J1-Pin_4) -> GPIO4
- J1 pad 5: Net-(J1-Pin_5) -> GPIO3
- J1 pad 8: Net-(J1-Pin_8) -> LED1
- J1 pad 9: Net-(J1-Pin_9) -> LED3
- J2 pad 15: Net-(J2-Pin_15) -> SW2
- J2 pad 16: Net-(J2-Pin_16) -> SW3
- U2 pad 10: Net-(J1-Pin_10) -> SW1
- U2 pad 12: Net-(J1-Pin_12) -> GPIO2
- U2 pad 13: Net-(J1-Pin_13) -> LED2
- U2 pad 14: Net-(J1-Pin_14) -> LED4
- U2 pad 15: Net-(J1-Pin_15) -> GPIO1
- U2 pad 16: Net-(J1-Pin_16) -> GPIO0
- U2 pad 19: Net-(J2-Pin_16) -> SW3
- U2 pad 20: Net-(J2-Pin_15) -> SW2
- U2 pad 4: Net-(J1-Pin_4) -> GPIO4
- U2 pad 5: Net-(J1-Pin_5) -> GPIO3
- U2 pad 8: Net-(J1-Pin_8) -> LED1
- U2 pad 9: Net-(J1-Pin_9) -> LED3
Routing:
- net VCC: track 0.00 -> 71.6 mm, vias 0 -> 66
- net SW1: track 17.3 -> 64.3 mm
- net Net-(D6-A): track 0.00 -> 29.7 mm
- net Net-(D8-A): track 0.00 -> 25.9 mm
- net SW2: track 17.3 -> 43.1 mm
- net Net-(D1-A): track 0.00 -> 22.5 mm
- net Net-(D5-A): track 0.00 -> 19.6 mm
- net +3V3: track 261.0 -> 279.6 mm
- net Net-(Q1-G): track 17.5 -> 33.8 mm
- net SW3: track 17.3 -> 33.1 mm
- net BUZZER: track 3.11 -> 17.9 mm
- net Net-(BZ1--): track 0.00 -> 14.7 mm
- net LED3: track 0.00 -> 11.0 mm
- net LED4: track 0.00 -> 11.0 mm
- net Net-(D7-A): track 0.00 -> 7.50 mm
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- added copper zone on B.Cu, net GND
- added copper zone on F.Cu, net GND
- removed copper zone on F.Cu, net Net-(D3-K)
Other:
- outline, holes or cut-outs redrawn
- board text added: "1"
- board text added: "10k"
- board text added: "1k"
- board text added: "2"
- board text added: "3"
- board text added: "3V3"
- board text added: "4"
- board text added: "ADC0"
- board text added: "ADC1"
- board text added: "Akizuki RP2040"
- board text added: "BATT"
- board text added: "Battery"
- board text added: "Buzzer"
- board text added: "Fuse"
- board text added: "GND"
- board text added: "GPIO0"
- board text added: "GPIO1"
- board text added: "GPIO2"
- board text added: "GPIO3"
- board text added: "GPIO4"
- board text added: "I2C"
- board text added: "Memo"
- board text added: "MotorDriver"
- board text added: "NPN"
- board text added: "PMOS"
- board text added: "PULLUP"
- board text added: "RX"
- board text added: "SCL"
- board text added: "SDA"
- board text added: "SIG"
- board text added: "TX"
- board text added: "UART0"
- board text added: "VCC"

Commit message: 最終修正
Parts:
- BZ1: value Buzzer -> PKM13EPYH4000-A0
- Q1: value Q_PMOS_GDS -> TJ60S04M3L
- SW1, SW3, SW4: value SW_Push_Dual -> TVGP01-G73BB
- SW2: value SW_Slide_DPDT -> IS-2235
Other:
- board text added: "MainBoard V1.1"

Commit message: 最終発注
Parts:
- R12, R7: value 10k -> 1k
Connections:
- net GPIO0 renamed GPIOA
- net GPIO1 renamed GPIOB
- net GPIO2 renamed GPIOC
- net GPIO3 renamed GPIOD
- net GPIO4 renamed GPIOE
Other:
- board text added: "GPIOA"
- board text added: "GPIOB"
- board text added: "GPIOC"
- board text added: "GPIOD"
- board text added: "GPIOE"
- board text removed: "GPIO0"
- board text removed: "GPIO1"
- board text removed: "GPIO2"
- board text removed: "GPIO3"
- board text removed: "GPIO4"

Commit message: これこそが最終発注
Other:
- board text added: "FreeSpace"
Changed lines of the file:
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@@
+		)
+	)
+	(gr_text "FreeSpace"
+		(at -26.5 -27 180)
+		(layer "B.SilkS" knockout)
+		(effects
+			(font
+				(size 1.5 1.5)
+				(thickness 0.3)
+				(bold yes)
+			)
+			(justify left bottom mirror)
 		)
 	)
